Commit message: Task2 Spawn robot in simulation

File: my_rb1_description/urdf/my_rb1_robot.urdf (robot description, URDF)
Before this commit: robot RB1, 6 links, 5 joints
Links:
- removed link back_caster_wheel
- removed link front_caster_wheel
- added link link_back_caster_wheel, mass 1; collision sphere radius=0.010; collision sphere radius=0.025
- added link link_front_caster_wheel, mass 1; collision sphere radius=0.010; collision sphere radius=0.025
Joints:
- joint back__caster_wheel: child back_caster_wheel -> link_back_caster_wheel
- joint front__caster_wheel: child front_caster_wheel -> link_front_caster_wheel
